Commit message: golden commit : Moveit works with python!

File: pkgs/duman_description/urdf/duman.urdf (robot description, URDF)
Before this commit: robot onshape, 10 links, 9 joints
Links:
- added link end_effector, mass 0.0; collision box size=0.001 0.001 0.001; visual box size=0.001 0.001 0.001
Joints:
- added joint end_effector_joint: type continuous, parent gripper_base, child end_effector, origin xyz=-0.1015213543711 0.0 0.0 rpy=0.0 2.419538725682435286e-17 1.3877787807813837993e-16, axis 1 0 0, limit effort=1 velocity=20
