Commit message: can move both arms at once, crazy work to come

File: pkgs/duman_description/urdf/duman_goat.urdf (robot description, URDF)
Before this commit: robot duman_arm, 16 links, 15 joints
Joints:
- joint left_elbow: limit lower=-3.141592653589793 upper=3.141592653589793 effort=10 velocity=10 -> lower=-1.57 upper=2.36 effort=4 velocity=4
- joint left_hip: limit lower=-3.141592653589793 upper=3.141592653589793 effort=10 velocity=10 -> lower=-0.78 upper=1.57 effort=4 velocity=4
- joint left_shoulder: limit lower=-3.141592653589793 upper=3.141592653589793 effort=10 velocity=10 -> lower=-1.57 upper=0.1 effort=4 velocity=4
- joint right_elbow: limit lower=-3.141592653589793 upper=3.141592653589793 effort=10 velocity=10 -> lower=-2.36 upper=1.57 effort=4 velocity=4
- joint right_hip: limit lower=-3.141592653589793 upper=3.141592653589793 effort=10 velocity=10 -> lower=-1.57 upper=0.78 effort=4 velocity=4
- joint right_shoulder: limit lower=-3.141592653589793 upper=3.141592653589793 effort=10 velocity=10 -> lower=-0.1 upper=1.57 effort=4 velocity=4

File: pkgs/protoman_moveit/config/onshape.urdf.xacro (robot description, xacro)
@@ -3,5 +3,5 @@
     <xacro:arg name="initial_positions_file" default="initial_positions.yaml" />
     <!-- Import onshape urdf file -->
-    <xacro:include filename="$(find duman_description)/urdf/duman.urdf" />
+    <xacro:include filename="$(find duman_description)/urdf/protoman.urdf" />
     <!-- Import control_xacro -->
     <xacro:include filename="onshape.ros2_control.xacro" />

Commit message: duman hardware

File: pkgs/duman_description/urdf/duman_goat.urdf (robot description, URDF)
Before this commit: robot duman_arm, 16 links, 15 joints
Joints:
- joint left_wrist1: limit lower=-3.141592653589793 upper=3.141592653589793 effort=10 velocity=10 -> lower=-1.57 upper=1.57 effort=4 velocity=4
- joint left_wrist2: limit lower=-3.141592653589793 upper=3.141592653589793 effort=10 velocity=10 -> lower=-1.57 upper=1.57 effort=4 velocity=4
- joint left_wrist3: limit lower=-3.141592653589793 upper=3.141592653589793 effort=10 velocity=10 -> lower=-1.57 upper=1.57 effort=4 velocity=4
- joint right_wrist1: limit lower=-3.141592653589793 upper=3.141592653589793 effort=10 velocity=10 -> lower=-1.57 upper=1.57 effort=4 velocity=4
- joint right_wrist2: limit lower=-3.141592653589793 upper=3.141592653589793 effort=10 velocity=10 -> lower=-1.57 upper=1.57 effort=4 velocity=4
- joint right_wrist3: limit lower=-3.141592653589793 upper=3.141592653589793 effort=10 velocity=10 -> lower=-1.57 upper=1.57 effort=4 velocity=4

Commit message: duman ik testing

File: pkgs/duman_description/urdf/duman_goat.urdf (robot description, URDF)
Before this commit: robot duman_arm, 16 links, 15 joints
Joints:
- joint wrist_to_ee_left: origin xyz=0 0 0.03 rpy=0 0 0 -> xyz=0 0 0.06 rpy=0 0 0
- joint wrist_to_ee_right: origin xyz=0 0 0.03 rpy=0 0 0 -> xyz=0 0 0.06 rpy=0 0 0

Commit message: depth camera added

File: pkgs/duman_description/urdf/duman_goat.urdf (robot description, URDF)
Before this commit: robot duman_arm, 16 links, 15 joints
Joints:
- joint wrist_to_ee_left: origin xyz=0 0 0.06 rpy=0 0 0 -> xyz=0 0 0.05 rpy=0 0 0
- joint wrist_to_ee_right: origin xyz=0 0 0.06 rpy=0 0 0 -> xyz=0 0 0.05 rpy=0 0 0

Commit message: obj detection in 3d space, handled ik failure

File: pkgs/duman_description/urdf/duman_goat.urdf (robot description, URDF)
Before this commit: robot duman_arm, 16 links, 15 joints
Links:
- added link camera_link
Joints:
- added joint base_to_camera: type fixed, parent base, child camera_link, origin xyz=0.04 0.05 0.695 rpy=-2.285 0 3.14
- joint left_elbow: origin xyz=-0.271178 0.0015 -0.0400426 rpy=2.52273e-15 4.22143e-15 -2.99867 -> xyz=-0.281178 0.0015 -0.0400426 rpy=2.52273e-15 4.22143e-15 -2.99867
- joint left_hip: origin xyz=0.279139 0.536574 0.432788 rpy=-1.5779 -0.0110701 1.57836 -> xyz=0.32 0.536574 0.432788 rpy=-1.5779 -0.0110701 1.57836
- joint left_shoulder: origin xyz=1.05013e-06 -0.0575174 -0.0580524 rpy=-1.5708 -1.36524e-15 -1.06156e-15 -> xyz=1.05013e-06 -0.0670174 -0.0580524 rpy=-1.5708 -1.36524e-15 -1.06156e-15
- joint right_elbow: origin xyz=0.271177 -1.38778e-17 -0.040137 rpy=2.01271e-15 -1.26764e-16 -3.40438e-16 -> xyz=0.281177 -1.38778e-17 -0.040137 rpy=2.01271e-15 -1.26764e-16 -3.40438e-16
- joint right_hip: origin xyz=-0.0574027 0.534054 0.430398 rpy=-1.56369 0.0110701 -1.56323 -> xyz=-0.0974027 0.534054 0.430398 rpy=-1.56369 0.0110701 -1.56323
- joint right_shoulder: origin xyz=1.05013e-06 -0.0575174 -0.0580524 rpy=-1.5708 8.46974e-16 2.26151e-17 -> xyz=1.05013e-06 -0.0670174 -0.0580524 rpy=-1.5708 8.46974e-16 2.26151e-17
- joint skeleton_to_base: origin xyz=-0.12 0.475 0 rpy=1.57 0 0 -> xyz=-0.115 0.49 0.03 rpy=1.57 0 0

Commit message: experiments

File: pkgs/duman_description/urdf/duman_goat.urdf (robot description, URDF)
Before this commit: robot duman_arm, 17 links, 16 joints
Joints:
- joint base_to_camera: origin xyz=0.04 0.05 0.695 rpy=-2.285 0 3.14 -> xyz=0.04 0.05 0.695 rpy=-2.22 0 3.14
